File: ESP32 Sensor.brd (EAGLE design)
At the start: 68.6 x 30.5 mm, 42 parts, among them J1 POWER_JACKPTH_LOCK, U1 TSL2572/TCS3472, U2 AP2112-3.3, U3 ESP32_WROOM32_SKINNY, U4 R-78E5.0-1.0, U5 BCR421, U6 BCR421, U7 MCP9700TT

Commit message: reva ordered
Parts:
- moved C4 28.2 mm to (40.2, 26.0)
- moved RST 27.8 mm to (36.1, 26.9), turned to 180 degrees
- moved R5 21.3 mm to (64.8, 2.54), turned to 270 degrees
- moved R6 20.9 mm to (62.2, 2.54), turned to 270 degrees
- moved R8 20.0 mm to (40.1, 24.4), turned to 0 degrees
- moved R12 19.4 mm to (34.8, 1.27)
- moved C3 7.52 mm to (34.3, 6.10), turned to 90 degrees
- moved R10 7.38 mm to (52.3, 2.29)
- moved U5 6.35 mm to (15.2, 24.1), turned to 270 degrees
- moved C7 5.71 mm to (42.4, 4.57), turned to 270 degrees
- moved D1 5.68 mm to (25.4, 15.2), turned to 180 degrees
- moved U6 5.24 mm to (16.5, 15.2), turned to 270 degrees
- moved R1 3.81 mm to (31.8, 14.0)
- moved R3 3.81 mm to (31.8, 15.6)
- moved D3 3.70 mm to (56.1, 2.29), turned to 270 degrees
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Connections:
- removed net A3_I39: U3.5
- removed net A4_IO36: U3.4
- removed net A5_IO4: U3.26
- removed net GPIO2: U3.24
- removed net IO12_A11: U3.14
- removed net IO14_A6: U3.13
- removed net IO15_A8: U3.23
- removed net IO16: U3.27
- removed net IO17: U3.28
- removed net IO21: U3.33
- removed net IO27_A10: U3.12
- removed net IO32_A7: U3.8
- removed net IO33_A9: U3.9
- removed net MISO: U3.31
- removed net MOSI: U3.30
- removed net SCK: U3.29
Routing:
- net GND: track 228.8 -> 0.00 mm, vias 2 -> 42
- net SDA: track 32.9 -> 49.9 mm
- net EN: track 50.0 -> 66.3 mm, vias 1 -> 0
- net 3.3V: track 88.1 -> 100.5 mm, vias 3 -> 2
- net VBUS: track 30.7 -> 41.5 mm
- net SCL: track 41.4 -> 49.7 mm
- net +12V: track 32.8 -> 40.5 mm
- net A1_DAC1: track 45.1 -> 38.8 mm, vias 0 -> 2
- net LED2_OUT: track 15.5 -> 9.31 mm
- net LED1_OUT: track 16.2 -> 10.3 mm
- net IO13_A12: track 8.30 -> 2.60 mm
- net A13_I35: track 22.3 -> 17.0 mm
- net A0_DAC2: track 44.1 -> 48.3 mm, vias 0 -> 2
- net RXD0: track 8.52 -> 10.4 mm
- net GPIO0: track 12.5 -> 14.2 mm
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- added copper zone on layer 1, net GND
- added copper zone on layer 16, net GND
Other:
- board text added: "2019"
- board text added: "570 LABS LLC"
- board text added: "A"
