File: ESP32 Sensor.sch (EAGLE design)
At the start: 42 parts, among them J1 POWER_JACKPTH_LOCK, U1 TSL2572/TCS3472, U2 AP2112-3.3, U3 ESP32_WROOM32_SKINNY, U4 R-78E5.0-1.0, U5 BCR421, U6 BCR421, U7 MCP9700TT

Commit message: reva ordered
Parts:
- R1, R3: MF (none) -> MF-RES-0603-100K
Connections:
- removed net A3_I39: U3.IO39/SEN_VN/A1_3
- removed net A4_IO36: U3.IO36/SEN_VP/A1_0
- removed net A5_IO4: U3.IO4/A2_0
- removed net GPIO2: U3.IO2/A2_2
- removed net IO12_A11: U3.IO12/A2_5
- removed net IO14_A6: U3.IO14/A2_6
- removed net IO15_A8: U3.IO15/A2_3
- removed net IO16: U3.IO16
- removed net IO17: U3.IO17
- removed net IO21: U3.IO21
- removed net IO27_A10: U3.IO27/A2_7
- removed net IO32_A7: U3.IO32/A1_4/X32P
- removed net IO33_A9: U3.IO33/A1_5/X32N
- removed net MISO: U3.IO19
- removed net MOSI: U3.IO18
- removed net SCK: U3.IO5
